File: Goggle-Display-Unit-Hat/Goggle-Display-Unit-Hat.kicad_sch (KiCad schematic)
At the start: 0 parts

Commit message: Boost converter and basic connector schematic work
Parts:
- added A1: Arduino_Giga_R1_WiFi_Shield, PCM_arduino-library:Arduino_Giga_R1_WiFi_Shield, symbol PCM_arduino-library:Arduino_Giga_R1_WiFi_Shield
- added C1, C8: 10uF, Capacitor_SMD:C_1206_3216Metric_Pad1.33x1.80mm_HandSolder, symbol Device:C
- added C2, C3: 1uF, Capacitor_SMD:C_0603_1608Metric_Pad1.08x0.95mm_HandSolder, symbol Device:C
- added C4, C7: 4.7uF, Capacitor_SMD:C_0603_1608Metric_Pad1.08x0.95mm_HandSolder, symbol Device:C
- added C5, C9: 0.1uF, Capacitor_SMD:C_0603_1608Metric_Pad1.08x0.95mm_HandSolder, symbol Device:C
- added C6: C, symbol Device:C
- added D1: MBR0530, Diode_SMD:D_SOD-123, symbol Device:D_Schottky
- added J1: 6871XX182122_687124182122, 6871XX182122_687124182122:687124182122, symbol 6871XX182122_687124182122:6871XX182122_687124182122
- added L1: LPS3015-103MRC, LPS3015-103MRC:IND_LPS3015-103MRC, symbol LPS3015-103MRC:LPS3015-103MRC
- added R1: 47K, Resistor_SMD:R_0603_1608Metric_Pad0.98x0.95mm_HandSolder, symbol Device:R
- added R2, R3: 5.1k, Resistor_SMD:R_0603_1608Metric_Pad0.98x0.95mm_HandSolder, symbol Device:R
- added R4: 910k, Resistor_SMD:R_0603_1608Metric_Pad0.98x0.95mm_HandSolder, symbol Device:R
- added R5: 10k, Resistor_SMD:R_0603_1608Metric_Pad0.98x0.95mm_HandSolder, symbol Device:R
- added U1: AP3012, Package_TO_SOT_SMD:SOT-23-5, symbol Regulator_Switching:AP3012
Connections:
- new net: D1.2 (A), L1.2, U1.1 (SW)
- new net: R1.2, R2.1, U1.3 (FB)
- new net +3.3V: C1.1, C2.1, L1.1, U1.5 (IN)
- new net GND: C1.2, C2.2, C3.2, R2.2, U1.2 (GND)
- new net VOLED: C3.1, D1.1 (K), R1.1
- new net VOLED_EN: A1.D6, U1.4 (~{SHDN})
Other:
- note added: "3.3V to 12.77v OLED Boost Supply"
